File: EnergyMonitoringSystem.kicad_pcb (KiCad board)
At the start: 6 copper layers, 170 x 117 mm, 205 parts, among them J201 USB_C_Receptacle_USB2.0_16P, J202 Screw_Terminal_01x02, J401 Conn_02x05_Counter_Clockwise, J402 Conn_02x05_Counter_Clockwise, J403 Conn_02x08_Counter_Clockwise, J501 Screw_Terminal_01x02, J502 Screw_Terminal_01x02, J503 Screw_Terminal_01x02, J504 Screw_Terminal_01x02, J505 Screw_Terminal_01x02, J506 Screw_Terminal_01x02, J601 DM3AT-SF-PEJM5_40_, J602 Screw_Terminal_01x03, Q201 STL6N3LLH6, SW401 SW_Push, SW402 SW_Push, U201 USBLC6-2P6, U202 STEF05SGR, U203 TCPP01-M12, U301 LDLN025M12R, U302 ST1PS02CQTR, U303 ST1PS02CQTR, U304 LM2664M6_NOPB, U401 STM32F103RGT6, U402 BLUENRG-M2SA, U501 ADS131M08IRSNR, U502 TSV914AIDR, U503 TSV914AIDR, U504 TSV914AIDR, U601 EMIF06-MSD02N16, U602 ADM2565EBRNZ, Y401 16MHz, Y402 32.768KHz

Commit message: all connections complete
Parts:
- moved H203 64.0 mm to (192.0, 147.0)
- moved FB601 37.5 mm to (191.3, 82.6), turned to 0 degrees
- moved D408 37.4 mm to (148.7, 104.1), turned to 180 degrees
- moved C419 36.0 mm to (145.6, 103.6), turned to 90 degrees
- moved C605 33.3 mm to (187.3, 83.5)
- moved R412 33.3 mm to (147.0, 100.4), turned to 90 degrees
- moved R413 33.1 mm to (148.7, 100.4), turned to 90 degrees
- moved C606 31.5 mm to (194.1, 83.4), turned to -90 degrees
- moved D402 30.2 mm to (115.6, 70.9)
- moved R411 29.8 mm to (150.3, 100.4), turned to 90 degrees
- moved SW401 29.8 mm to (119.1, 67.3)
- moved C401 29.4 mm to (113.3, 67.8), turned to -90 degrees
- moved R601 28.9 mm to (187.5, 92.4)
- moved D407 28.9 mm to (155.2, 58.9), turned to -90 degrees
- moved D406 25.6 mm to (158.2, 58.9), turned to -90 degrees
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Connections:
- J403 pad 20: unconnected-(J403-Pin_20-Pad20) -> ADS_DRDY
Routing:
- net +DCDC_2: track 8.10 -> 270.1 mm, vias 0 -> 5
- net UART_RTS_485: track 0.00 -> 127.9 mm, vias 0 -> 2
- net GND: track 290.0 -> 410.6 mm, vias 85 -> 111
- net UART_INV_485: track 0.00 -> 118.5 mm, vias 0 -> 4
- net UART_TX_485: track 0.00 -> 117.0 mm, vias 0 -> 2
- net UART_RX_485: track 0.00 -> 111.0 mm, vias 0 -> 2
- net DCDC_2_EN: track 2.09 -> 104.7 mm, vias 0 -> 4
- net SD_DETECT: track 0.00 -> 93.8 mm, vias 0 -> 5
- net GPIO1_Output: track 0.00 -> 86.3 mm, vias 0 -> 1
- net /uC/BLE_SPI_CS: track 74.1 -> 142.9 mm, vias 2 -> 3
- net /uC/SPI2_MOSI: track 57.8 -> 125.0 mm, vias 2 -> 3
- net /uC/NRST: track 0.00 -> 66.1 mm, vias 0 -> 2
- net I2C1_SDA: track 0.00 -> 59.1 mm, vias 0 -> 1
- net ADS_DIN_uC_DOUT: track 31.5 -> 89.0 mm, vias 0 -> 2
- net I2C1_SCL: track 0.00 -> 57.2 mm, vias 0 -> 1
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Other:
- board size 170 x 117 mm -> 170 x 114.4 mm
- rule pad_to_mask_clearance: 0.08 -> 0
