File: adc.kicad_sch (KiCad schematic)
At the start: 68 parts, among them J601 Screw_Terminal_01x02, J602 Screw_Terminal_01x02, J603 Screw_Terminal_01x02, J604 Screw_Terminal_01x02, J605 Screw_Terminal_01x02, J606 Screw_Terminal_01x02, U601 ADS131M08IRSNR, U602 TSV911ILT, U603 TSV911ILT, U604 TSV911ILT

Commit message: minor formatting updates
Parts:
- renumbered C603 to C602, C604 to C603, C606 to C604, C607 to C605, C609 to C606, C602 to C607, C605 to C608, C608 to C609, C614 to C610, C616 to C611, C618 to C612, C615 to C613, C617 to C614, C619 to C615, C611 to C616, C612 to C617, C610 to C618, C613 to C619, R605 to R601, R612 to R602, R619 to R603, R601 to R604, R608 to R605, R615 to R606, R633 to R607, R636 to R608, R639 to R609, R602 to R610, R609 to R611, R616 to R612, R603 to R613, R610 to R614, R617 to R615, R632 to R616, R635 to R617, R638 to R618, R606 to R619, R613 to R620, R620 to R621, R604 to R622, R607 to R623, R611 to R624, R614 to R625, R618 to R626, R621 to R627, R634 to R629, R637 to R630, R623 to R631, R624 to R632, R626 to R633, R629 to R634, R631 to R635, R622 to R636, R625 to R637, R627 to R638, R630 to R639, U602 to U601, U603 to U602, U604 to U603, U601 to U604

Commit message: validation BOM
Parts:
- R616, R617, R618: Distributor_Link https://www.mouser.com/ProductDetail/Panasonic/ERJ-S03F1502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 -> https://www.mouser.com/ProductDetail/Panasonic/ERJ-3EKF1502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; Manufacturer_Part_Number ERJ-S03F1502V -> ERJ-3EKF1502V
Changed lines of the file:
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@@
 			)
 		)
-		(property "Distributor_Link" "https://www.mouser.com/ProductDetail/Panasonic/ERJ-S03F1502V?qs=Zyl8A9hlmJqFaE%2FSdjcX1A%3D%3D"
+		(property "Distributor_Link" "https://www.mouser.com/ProductDetail/Panasonic/ERJ-3EKF1502V?qs=H7k1u0Mp9JTF6x646045AQ%3D%3D"
 			(at 85.09 300.99 0)
 			(effects
@@
 			)
 		)
-		(property "Manufacturer_Part_Number" "ERJ-S03F1502V "
+		(property "Manufacturer_Part_Number" "ERJ-3EKF1502V"
 			(at 85.09 300.99 0)
 			(effects
@@
 			)
 		)
-		(property "Distributor_Link" "https://www.mouser.com/ProductDetail/Panasonic/ERJ-S03F1502V?qs=Zyl8A9hlmJqFaE%2FSdjcX1A%3D%3D"
+		(property "Distributor_Link" "https://www.mouser.com/ProductDetail/Panasonic/ERJ-3EKF1502V?qs=H7k1u0Mp9JTF6x646045AQ%3D%3D"
 			(at 85.09 231.14 0)
 			(effects
@@
 			)
 		)
-		(property "Manufacturer_Part_Number" "ERJ-S03F1502V "
+		(property "Manufacturer_Part_Number" "ERJ-3EKF1502V"
 			(at 85.09 231.14 0)
 			(effects
@@
 			)
 		)
-		(property "Distributor_Link" "https://www.mouser.com/ProductDetail/Panasonic/ERJ-S03F1502V?qs=Zyl8A9hlmJqFaE%2FSdjcX1A%3D%3D"
+		(property "Distributor_Link" "https://www.mouser.com/ProductDetail/Panasonic/ERJ-3EKF1502V?qs=H7k1u0Mp9JTF6x646045AQ%3D%3D"
 			(at 87.63 372.11 0)
 			(effects
@@
 			)
 		)
-		(property "Manufacturer_Part_Number" "ERJ-S03F1502V "
+		(property "Manufacturer_Part_Number" "ERJ-3EKF1502V"
 			(at 87.63 372.11 0)
 			(effects
