File: uCMain.kicad_sch (KiCad schematic)
At the start: 74 parts, among them J401 Conn_02x05_Counter_Clockwise, SW401 SW_Push, SW402 SW_Push, U401 STM32H745ZGT6, Y401 Crystal_GND24, Y402 32.768KHz

Commit message: minor design improvements
Parts:
- C412, C413, C428, C435: Manufacturer_Part_Number 04023C104KAT2A -> KGM05AR51A225KH
Changed lines of the file:
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@@
 			)
 		)
-		(property "Manufacturer_Part_Number" "04023C104KAT2A"
+		(property "Manufacturer_Part_Number" "KGM05AR51A225KH"
 			(at 285.75 203.2 0)
 			(effects
@@
 			)
 		)
-		(property "Manufacturer_Part_Number" "04023C104KAT2A"
+		(property "Manufacturer_Part_Number" "KGM05AR51A225KH"
 			(at 278.13 203.2 0)
 			(effects
@@
 			)
 		)
-		(property "Manufacturer_Part_Number" "04023C104KAT2A"
+		(property "Manufacturer_Part_Number" "KGM05AR51A225KH"
 			(at 195.58 130.81 0)
 			(effects
@@
 			)
 		)
-		(property "Manufacturer_Part_Number" "04023C104KAT2A"
+		(property "Manufacturer_Part_Number" "KGM05AR51A225KH"
 			(at 195.58 135.89 0)
 			(effects

Commit message: solder bridge fixed
Parts:
- JP401, JP402, JP403, JP406, JP408: footprint Jumper:SolderJumper-2_P1.3mm_Bridged_RoundedPad1.0x1.5mm -> Jumper:SolderJumper-2_P1.3mm_Open_RoundedPad1.0x1.5mm
Changed lines of the file:
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@@
 			)
 		)
-		(property "Footprint" "Jumper:SolderJumper-2_P1.3mm_Bridged_RoundedPad1.0x1.5mm"
+		(property "Footprint" "Jumper:SolderJumper-2_P1.3mm_Open_RoundedPad1.0x1.5mm"
 			(at 212.09 166.37 0)
 			(effects
@@
 			)
 		)
-		(property "Footprint" "Jumper:SolderJumper-2_P1.3mm_Bridged_RoundedPad1.0x1.5mm"
+		(property "Footprint" "Jumper:SolderJumper-2_P1.3mm_Open_RoundedPad1.0x1.5mm"
 			(at 212.09 123.19 0)
 			(effects
@@
 			)
 		)
-		(property "Footprint" "Jumper:SolderJumper-2_P1.3mm_Bridged_RoundedPad1.0x1.5mm"
+		(property "Footprint" "Jumper:SolderJumper-2_P1.3mm_Open_RoundedPad1.0x1.5mm"
 			(at 212.09 120.65 0)
 			(effects
@@
 			)
 		)
-		(property "Footprint" "Jumper:SolderJumper-2_P1.3mm_Bridged_RoundedPad1.0x1.5mm"
+		(property "Footprint" "Jumper:SolderJumper-2_P1.3mm_Open_RoundedPad1.0x1.5mm"
 			(at 199.39 111.76 0)
 			(effects
@@
 			)
 		)
-		(property "Footprint" "Jumper:SolderJumper-2_P1.3mm_Bridged_RoundedPad1.0x1.5mm"
+		(property "Footprint" "Jumper:SolderJumper-2_P1.3mm_Open_RoundedPad1.0x1.5mm"
 			(at 212.09 139.7 0)
 			(effects
